Commit message: Added basic gazebo diff control

File: src/lookout_tower/description/robot.urdf.xacro (robot description, xacro)
@@ -1,4 +1,5 @@
 <?xml version="1.0"?>
 <robot xmlns:xacro="http://www.ros.org/wiki/xacro" name="robot">
-    <xacro:include filename="robot_core.xacro" />
+    <xacro:include filename="robot_core.xacro"/>
+    <xacro:include filename="gazebo_control.xacro"/>
 </robot>

File: src/lookout_tower/description/robot_core.xacro (robot description, xacro)
@@ -1,4 +1,7 @@
 <?xml version="1.0"?>
 <robot xmlns:xacro="http://www.ros.org/wiki/xacro">
+    <!-- PROPERTIES -->
+    <xacro:property name="pi" value="3.141592653589793"/>
+    <!-- MATERIALS (Colors) -->
     <material name="black">
         <color rgba="0 0 0 1"/>
@@ -36,4 +39,7 @@
         </collision>
     </link>
+    <gazebo reference="chassis">
+        <material>Gazebo/Black</material>
+    </gazebo>
     <!-- FRONT LEFT WHEEL LINK -->
     <joint name="front_left_wheel_joint" type="continuous">
@@ -44,4 +50,9 @@
     </joint>
     <link name="front_left_wheel">
+        <inertial>
+        <origin xyz="0 0 0" rpy="0 0 0"/>
+        <mass value="0.1"/>
+        <inertia ixx="0.0057" ixy="0.0" ixz="0.0" iyy="0.0057" iyz="0.0" izz="0.00072"/>
+        </inertial>
         <visual>
             <geometry>
@@ -50,5 +61,16 @@
             <material name="blue"/>
         </visual>
+        <collision>
+        <origin xyz="0 0 0" rpy="0 0 0"/>
+            <geometry>
+                <cylinder radius="0.12" length="0.08"/>
+            </geometry>
+        </collision>
     </link>
+    <gazebo reference="front_left_wheel">
+        <material>Gazebo/Blue</material>
+        <mu1 value="0.001"/> <!-- PLACEHOLDER BEFORE ACKERMANN STEERING -->
+        <mu2 value="0.001"/> <!-- PLACEHOLDER BEFORE ACKERMANN STEERING -->
+    </gazebo>
     <!-- FRONT RIGHT WHEEL LINK -->
     <joint name="front_right_wheel_joint" type="continuous">
@@ -56,7 +78,12 @@
         <child link="front_right_wheel"/>
         <origin xyz="0.2 -0.24 0" rpy="${pi/2} 0 0"/>
-        <axis xyz="0 0 -1"/>
+        <axis xyz="0 0 1"/>
     </joint>
     <link name="front_right_wheel">
+        <inertial>
+        <origin xyz="0 0 0" rpy="0 0 0"/>
+        <mass value="0.1"/>
+        <inertia ixx="0.0057" ixy="0.0" ixz="0.0" iyy="0.0057" iyz="0.0" izz="0.00072"/>
+        </inertial>
         <visual>
             <geometry>
@@ -65,5 +92,16 @@
             <material name="blue"/>
         </visual>
+        <collision>
+        <origin xyz="0 0 0" rpy="0 0 0"/>
+            <geometry>
+                <cylinder radius="0.12" length="0.08"/>
+            </geometry>
+        </collision>
     </link>
+    <gazebo reference="front_right_wheel">
+        <material>Gazebo/Blue</material>
+        <mu1 value="0.001"/> <!-- PLACEHOLDER BEFORE ACKERMANN STEERING -->
+        <mu2 value="0.001"/> <!-- PLACEHOLDER BEFORE ACKERMANN STEERING -->
+    </gazebo>
     <!-- BACK LEFT WHEEL LINK -->
     <joint name="back_left_wheel_joint" type="continuous">
@@ -71,7 +109,12 @@
         <child link="back_left_wheel"/>
         <origin xyz="-0.2 0.24 0" rpy="${pi/2} 0 0"/>
-        <axis xyz="0 0 1"/>
+        <axis xyz="0 0 -1"/>
     </joint>
     <link name="back_left_wheel">
+        <inertial>
+        <origin xyz="0 0 0" rpy="0 0 0"/>
+        <mass value="0.1"/>
+        <inertia ixx="0.0057" ixy="0.0" ixz="0.0" iyy="0.0057" iyz="0.0" izz="0.00072"/>
+        </inertial>
         <visual>
             <geometry>
@@ -80,5 +123,14 @@
             <material name="blue"/>
         </visual>
+        <collision>
+        <origin xyz="0 0 0" rpy="0 0 0"/>
+            <geometry>
+                <cylinder radius="0.12" length="0.08"/>
+            </geometry>
+        </collision>
     </link>
+    <gazebo reference="back_left_wheel">
+        <material>Gazebo/Blue</material>
+    </gazebo>
     <!-- BACK RIGHT WHEEL LINK -->
     <joint name="back_right_wheel_joint" type="continuous">
@@ -89,4 +141,9 @@
     </joint>
     <link name="back_right_wheel">
+        <inertial>
+        <origin xyz="0 0 0" rpy="0 0 0"/>
+        <mass value="0.1"/>
+        <inertia ixx="0.0057" ixy="0.0" ixz="0.0" iyy="0.0057" iyz="0.0" izz="0.00072"/>
+        </inertial>
         <visual>
             <geometry>
@@ -95,4 +152,13 @@
             <material name="blue"/>
         </visual>
+        <collision>
+        <origin xyz="0 0 0" rpy="0 0 0"/>
+            <geometry>
+                <cylinder radius="0.12" length="0.08"/>
+            </geometry>
+        </collision>
     </link>
+    <gazebo reference="back_right_wheel">
+        <material>Gazebo/Blue</material>
+    </gazebo>
 </robot>
