Commit message: More robust pose estimation based on multi color wheels

File: src/lookout_tower/description/robot_core.xacro (robot description, xacro)
@@ -69,5 +69,5 @@
     </link>
     <gazebo reference="front_left_wheel">
-        <material>Gazebo/Blue</material>
+        <material>Gazebo/Red</material>
         <mu1 value="0.001"/> <!-- PLACEHOLDER BEFORE ACKERMANN STEERING -->
         <mu2 value="0.001"/> <!-- PLACEHOLDER BEFORE ACKERMANN STEERING -->
@@ -100,5 +100,5 @@
     </link>
     <gazebo reference="front_right_wheel">
-        <material>Gazebo/Blue</material>
+        <material>Gazebo/Red</material>
         <mu1 value="0.001"/> <!-- PLACEHOLDER BEFORE ACKERMANN STEERING -->
         <mu2 value="0.001"/> <!-- PLACEHOLDER BEFORE ACKERMANN STEERING -->

Commit message: a* algorithm implemented, but not working with dynamic map just yet

File: src/lookout_tower/description/robot_core.xacro (robot description, xacro)
@@ -42,4 +42,33 @@
         <material>Gazebo/Black</material>
     </gazebo>
+    <!-- STEERING LINK (For Ackermann steering)
+    <joint name="steering_joint" type="continuous">
+        <parent link="base_link"/>
+        <child link="steering_link"/>
+        <origin xyz="0 0 0" rpy="0 0 0"/>
+        <axis xyz="0 1 0"/>
+        <limit lower="-0.418879" upper="0.418879" velocity="1.0"/>
+        <dynamics damping="0.01"/>
+    </joint>
+    <link name="steering_link">
+        <inertial>
+            <origin xyz="0 0 0" rpy="0 0 0"/>
+            <mass value="0.01"/>
+            <inertia ixx="0.0001" ixy="0.0" ixz="0.0" iyy="0.0001" iyz="0.0" izz="0.0001"/>
+        </inertial>
+        <visual>
+            <origin xyz="0 0 0" rpy="0 0 0"/>
+            <geometry>
+                <box size="0.01 0.01 0.01"/>
+            </geometry>
+            <material name="black"/>
+        </visual>
+        <collision>
+            <origin xyz="0 0 0" rpy="0 0 0"/>
+            <geometry>
+                <box size="0.01 0.01 0.01"/>
+            </geometry>
+        </collision>
+    </link> -->
     <!-- FRONT LEFT WHEEL LINK -->
     <joint name="front_left_wheel_joint" type="continuous">
